File: PCBs/R0.1 Mainboard/Sizzle mainboard/Sizzle mainboard.kicad_sch (KiCad schematic)
At the start: 36 parts, among them J1 X Stepper, J2 Screen, J3 USB_C_Receptacle_USB2.0_16P, J4 Debug, J5 Z Stepper, J6 Y Stepper, J7 UV light, Q1 Q_NMOS_GSD, SW1 SW_Push, U1 STM32F401RCTx, U2 USBLC6-2SC6, U3 X Driver, U4 Y Driver, U5 Z Driver, U6 AP2127R-3.3, U7 MAX1659ESA, Y1 48MHz

Commit message: buck converters
Parts:
- removed D1, D2: D, symbol Device:D
- removed U6: AP2127R-3.3, Package_TO_SOT_SMD:SOT-89-3, symbol Regulator_Linear:AP2127R-3.3
- removed U7: MAX1659ESA, Package_SO:SOIC-8_3.9x4.9mm_P1.27mm, symbol Regulator_Linear:MAX1659ESA
- added C14: 180uF, symbol Device:C
- added C15: 470uF, symbol Device:C
- added D1, D2: D_Schottky, symbol Device:D_Schottky
- added J8: Power, symbol Connector_Generic:Conn_01x02
- added L1, L2: 68uh/2A, symbol Device:L
- added R4: 1k, symbol Device:R
- added R5: 10k, symbol Device:R
- added U6: XL1509-3.3, Package_SO:SOIC-8_3.9x4.9mm_P1.27mm, symbol Regulator_Switching:XL1509-3.3
- added U7: XL1509-5.0, Package_SO:SOIC-8_3.9x4.9mm_P1.27mm, symbol Regulator_Switching:XL1509-5.0
- C10: value 1uF -> 470uF
- C11: value 1uF -> 180uF
- C12: value 0.1uF -> 105
- C13: value 10uF -> 105
Connections:
- net +3.3V: now also J4.1 (Pin_1); no longer C11.1
- net +5V: no longer C13.1
- net GND: now also C14.2, C15.2, D1.2 (A), D2.2 (A), J8.2 (Pin_2), R5.2, U6.4 (~{EN}), U6.5 (GND), U6.6 (GND), U6.7 (GND), U6.8 (GND), U7.4 (~{EN}), U7.5 (GND), U7.6 (GND), U7.7 (GND), U7.8 (GND)
- net UV_LIGHT: now also R4.1, R5.1; no longer Q1.1 (G)
- net VBUS: no longer C10.1
- net VDD renamed +12V
- net +12V: now also C10.1, C13.1, C15.1, J8.1 (Pin_1), U6.1 (VIN), U7.1 (VIN); no longer J4.1 (Pin_1)
- new net: D1.1 (K), L1.1, U6.2 (OUT)
- new net: C11.1, L1.2, U6.3 (FB)
- new net: D2.1 (K), L2.1, U7.2 (OUT)
- new net: C14.1, L2.2, U7.3 (FB)
- new net: Q1.1 (G), R4.2
Other:
- moved on the sheet: J7, Q1

Commit message: Cleanup schematic, add buck converter, add other sensors
Parts:
- removed D1, D2: D_Schottky, symbol Device:D_Schottky
- removed U6: XL1509-3.3, Package_SO:SOIC-8_3.9x4.9mm_P1.27mm, symbol Regulator_Switching:XL1509-3.3
- removed U7: XL1509-5.0, Package_SO:SOIC-8_3.9x4.9mm_P1.27mm, symbol Regulator_Switching:XL1509-5.0
- added C13: 0.1uF, symbol Device:C
- added J10: Screen, symbol Connector_Generic:Conn_01x04
- added J9: Power, symbol Connector_Generic:Conn_01x02
- added L1: 4.7uH, symbol Device:L
- added U6: AP63203WU, Package_TO_SOT_SMD:TSOT-23-6, symbol Regulator_Switching:AP63203WU
- C10: value 470uF -> 0.1uF
- C11: value 180uF -> 1uF
- C12: value 105 -> 10uF
- C14: value 180uF -> 22uF
- C15: value 470uF -> 22uF
- C8, C9: value 0.1uF -> C
- J8: value Power -> Spindle Relay
- R4: value 1k -> 200R
- Y1: value 48MHz -> 25MHz
Connections:
- net +5V is gone; now on net +12V: Q1.2 (S), U3.8 (VCC), U4.8 (VCC), U5.8 (VCC)
- net +12V: now also J9.1 (Pin_1), U6.2 (EN), U6.3 (IN); no longer C10.1, C13.1, C15.1, J8.1 (Pin_1)
- net +3.3V: now also C11.1, C14.1, C15.1, U1.13 (VREF+), J10.1 (Pin_1), L1.2, U6.1 (FB)
- net GND: now also R5.1, J9.2 (Pin_2), U6.4 (GND); no longer C13.2, R5.2
- net UV_LIGHT: now also R5.2; no longer R5.1, U1.50 (PA15)
- net X_DIAG: no longer U1.41 (PA8)
- net X_DIR: no longer U1.20 (PA4)
- net X_INDEX: no longer U1.23 (PA7)
- net X_SPREAD: no longer U1.22 (PA6)
- net X_STEP: no longer U1.21 (PA5)
- net Y_DIAG: no longer U1.43 (PA10)
- net Y_DIR: no longer U1.26 (PB0)
- net Y_INDEX: no longer U1.42 (PA9)
- net Y_SPREAD: no longer U1.28 (PB2)
- net Y_STEP: no longer U1.27 (PB1)
- net Z_DIAG: no longer U1.33 (PB12)
- net Z_DIR: no longer U1.59 (PB7)
- net Z_INDEX: no longer U1.29 (PB10)
- net Z_SPREAD: no longer U1.62 (PB9)
- net Z_STEP: no longer U1.61 (PB8)
- net at L1.2: no longer C11.1
- net at U1.30 (VCAP1): now also C10.1
- net IR_SDA: now reaches U1.40 (PC9)
- net IR_SDA: now also J10.2 (Pin_2)
- net at L2.2: no longer C14.1
- new net: C13.1, U6.5 (SW)
- new net: C13.2, L1.1, U6.6 (BST)
- new net IR_SCL: J10.3 (Pin_3), U1.41 (PA8)
- new net SPINDLE_RELAY: J8.1 (Pin_1)
Other:
- title: (none) -> Sizzle CNC Mainboard
- moved on the sheet: C1, C2, C3, C4, C5, C6, C7, C8, C9, J1, J2, J3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

Commit message: Fix file, add .DS_Store to global gitignore
Parts:
- removed C13: 0.1uF, symbol Device:C
- removed J10: Screen, symbol Connector_Generic:Conn_01x04
- removed J9: Power, symbol Connector_Generic:Conn_01x02
- removed L1: 4.7uH, symbol Device:L
- removed U6: AP63203WU, Package_TO_SOT_SMD:TSOT-23-6, symbol Regulator_Switching:AP63203WU
- added D1, D2: D_Schottky, symbol Device:D_Schottky
- added U6: XL1509-3.3, Package_SO:SOIC-8_3.9x4.9mm_P1.27mm, symbol Regulator_Switching:XL1509-3.3
- added U7: XL1509-5.0, Package_SO:SOIC-8_3.9x4.9mm_P1.27mm, symbol Regulator_Switching:XL1509-5.0
- C10: value 0.1uF -> 470uF
- C11: value 1uF -> 180uF
- C12: value 10uF -> 105
- C14: value 22uF -> 180uF
- C15: value 22uF -> 470uF
- C8, C9: value C -> 0.1uF
- J8: value Spindle Relay -> Power
- R4: value 200R -> 1k
- Y1: value 25MHz -> 48MHz
Connections:
- net IR_SCL is gone; now on net X_DIAG: U1.41 (PA8)
- net SPINDLE_RELAY is gone; now on net +12V: J8.1 (Pin_1)
- net +12V: now also C10.1, C13.1, C15.1, U6.1 (VIN), U7.1 (VIN); no longer Q1.2 (S), U3.8 (VCC), U4.8 (VCC), U5.8 (VCC)
- net +3.3V: no longer C11.1, C14.1, C15.1, U1.13 (VREF+)
- net GND: now also C13.2, R5.2, D1.2 (A), D2.2 (A), U6.4 (~{EN}), U6.5 (GND), U6.6 (GND), U6.7 (GND), U6.8 (GND), U7.4 (~{EN}), U7.5 (GND), U7.6 (GND), U7.7 (GND), U7.8 (GND); no longer R5.1
- net UV_LIGHT: now also R5.1, U1.50 (PA15); no longer R5.2
- net X_DIR: now also U1.20 (PA4)
- net X_INDEX: now also U1.23 (PA7)
- net X_SPREAD: now also U1.22 (PA6)
- net X_STEP: now also U1.21 (PA5)
- net Y_DIAG: now also U1.43 (PA10)
- net Y_DIR: now also U1.26 (PB0)
- net Y_INDEX: now also U1.42 (PA9)
- net Y_SPREAD: now also U1.28 (PB2)
- net Y_STEP: now also U1.27 (PB1)
- net Z_DIAG: now also U1.33 (PB12)
- net Z_DIR: now also U1.59 (PB7)
- net Z_INDEX: now also U1.29 (PB10)
- net Z_SPREAD: now also U1.62 (PB9)
- net Z_STEP: now also U1.61 (PB8)
- net at L1.1: now also D1.1 (K), U6.2 (OUT)
- net at L1.2: now also C11.1, U6.3 (FB)
- net at U1.30 (VCAP1): no longer C10.1
- net at L2.1: now also D2.1 (K), U7.2 (OUT)
- net at L2.2: now also C14.1, U7.3 (FB)
- net IR_SDA: no longer names the net of U1.40 (PC9)
- new net +5V: Q1.2 (S), U3.8 (VCC), U4.8 (VCC), U5.8 (VCC)
Other:
- title: Sizzle CNC Mainboard -> (none)
- moved on the sheet: C1, C2, C3, C4, C5, C6, C7, C8, C9, J1, J2, J3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
